File: Carte_moteur/Carte_moteur.kicad_pcb (KiCad board)
At the start: 2 copper layers, 72.6 x 73.7 mm, 122 parts, among them J101 Conn_02x04_Top_Bottom, J103 Conn_01x02, J104 Conn_01x07, J105 Conn_01x02, J106 Conn_01x07, J201 Conn_01x05_Pin, J202 Conn_01x04_Pin, J301 Conn_01x05_Pin, J302 Conn_01x04_Pin, J401 Conn_01x05_Pin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

Commit message: fuck. Fuck fuck. Fuck Fuck Fuck. FUUCKING FUCK
Parts:
- added R619: 1k, Resistor_SMD:R_0603_1608Metric_Pad0.98x0.95mm_HandSolder, B.Cu at (140.0, 99.8)
- C201, C301, C401: value C -> 47uF
- C202, C302, C402, C508, C601, C602: value C -> 10uF
- C503, C504, C505, C506, C603, C604, C606, C607: value C -> 100nF
- C608, C609: value C -> 20pF
- J101: value Conn_02x04_Top_Bottom -> 1053141308
- J104, J106: value Conn_01x07 -> KK-254_AE-6410-07A
- J201, J301, J401: value Conn_01x05_Pin -> KK-254_AE-6410-05A
- J202, J302, J402: value Conn_01x04_Pin -> KK-254_AE-6410-04A
- J602: value USB_B_Mini -> 629105150521
- R101, R102, R103, R104, R105, R518, R601, R602: value R_US -> 10R
- R201, R204, R207, R301, R304, R307, R401, R404, R407, R603: value R_US -> 0R
- R202, R302, R402, R613: value R_US -> DNP
- R203, R206, R210, R211, R212, R303, R306, R403, R406, R510, R523, R524, R525, R526, R527, R528, R614: value R_US -> 10k
- R511, R611: value R_US -> 100R
- R512, R513, R514, R515, R516, R517, R615, R616, R617, R618: value R_US -> 1k
- R519: value R_US -> 10K
- R605: value 36k -> 33k
- R607, R608, R620: value R_US -> 4k7
- R621: value R_US -> 22k
- U603: value STM32F103CBTx -> STM32F103CBT6
- Y601: value Crystal_GND24 -> 8MHz
Connections:
- Q601 pad 2: Net-(J602-D+) -> Net-(Q601-E)
Routing:
- net Net-(J602-D+): track 10.8 -> 6.80 mm
- net Net-(Q601-E): track 0.00 -> 1.72 mm
