File: Carte_moteur/stlink.kicad_sch (KiCad schematic)
At the start: 36 parts, among them J601 Conn_01x06_Pin, J602 USB_B_Mini, Q601 MMBTA44, U601 ECMF02-2AMX6, U602 LD1117S33TR_SOT223, U603 STM32F103CBTx, Y601 Crystal_GND24

Commit message: changed pwr connector
Connections:
- no-connect marks 0 -> 15
Changed lines of the file:
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@@
 	)
 	(junction
+		(at 129.54 168.91)
+		(diameter 0)
+		(color 0 0 0 0)
+	)
+	(junction
 		(at 172.72 29.21)
 		(diameter 0)
@@
 		(color 0 0 0 0)
 	)
+	(no_connect
+		(at 187.96 83.82)
+	)
+	(no_connect
+		(at 187.96 91.44)
+	)
+	(no_connect
+		(at 187.96 78.74)
+	)
+	(no_connect
+		(at 152.4 60.96)
+	)
+	(no_connect
+		(at 187.96 106.68)
+	)
+	(no_connect
+		(at 152.4 43.18)
+	)
+	(no_connect
+		(at 187.96 63.5)
+	)
+	(no_connect
+		(at 187.96 81.28)
+	)
+	(no_connect
+		(at 187.96 76.2)
+	)
+	(no_connect
+		(at 187.96 96.52)
+	)
+	(no_connect
+		(at 152.4 50.8)
+	)
+	(no_connect
+		(at 187.96 93.98)
+	)
+	(no_connect
+		(at 187.96 88.9)
+	)
+	(no_connect
+		(at 187.96 86.36)
+	)
+	(no_connect
+		(at 187.96 71.12)
+	)
 	(wire
 		(pts
@@
 	(wire
 		(pts
+			(xy 129.54 168.91) (xy 124.46 168.91)
+		)
+		(stroke
+			(width 0)
+			(type default)
+		)
+	)
+	(wire
+		(pts
 			(xy 50.8 76.2) (xy 60.96 76.2)
 		)
@@
 	(wire
 		(pts
-			(xy 135.89 168.91) (xy 124.46 168.91)
+			(xy 135.89 168.91) (xy 129.54 168.91)
 		)
 		(stroke
@@
 					(unit 1)
 				)
+			)
+		)
+	)
+	(symbol
+		(lib_id "power:PWR_FLAG")
+		(at 129.54 168.91 0)
+		(unit 1)
+		(exclude_from_sim no)
+		(in_bom yes)
+		(on_board yes)
+		(dnp no)
+		(fields_autoplaced yes)
+		(property "Reference" "#FLG0601"
+			(at 129.54 167.005 0)
+			(effects
+				(font
+					(size 1.27 1.27)
+				)
+				(hide yes)
+			)
+		)
+		(property "Value" "PWR_FLAG"
+			(at 129.54 163.83 0)
+			(effects
+				(font
+					(size 1.27 1.27)
+				)
+			)
+		)
+		(property "Footprint" ""
+			(at 129.54 168.91 0)
+			(effects
+				(font
+					(size 1.27 1.27)
+				)
+				(hide yes)
+			)
+		)
+		(property "Datasheet" "~"
+			(at 129.54 168.91 0)
+			(effects
+				(font
+					(size 1.27 1.27)
+				)
+				(hide yes)
+			)
+		)
+		(property "Description" "Special symbol for telling ERC where power comes from"
+			(at 129.54 168.91 0)
+			(effects
+				(font
+					(size 1.27 1.27)
+				)
+				(hide yes)
+			)
+		)
+		(pin "1"
+		)
+		(instances
+			(project ""
+				(path "/5d858058-eb89-4613-a7ba-0652b9f0936c/a0d73204-6cde-434c-a6b9-1c87c98088a0"
+					(reference "#FLG0601")
+					(unit 1)
+				)

Commit message: update motor board values
Parts:
- C601, C602: value C -> 10uF
- C603, C604, C606, C607: value C -> 100nF
- C608, C609: value C -> 20pF
- J602: value USB_B_Mini -> 629105150521
- R601, R602, R603: value R_US -> 0R
- R605: value 36k -> 33k
- R607, R608: value R_US -> 4k7
- R611: value R_US -> 100R
- R613: value R_US -> DNP
- R614: value R_US -> 10k
- R615, R616: value R_US -> 1k
- U603: value STM32F103CBTx -> STM32F103CBT6
- Y601: value Crystal_GND24 -> 8MHz
Changed lines of the file:
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@@
 		(fields_autoplaced yes)
 		(property "Reference" "R607"
-			(at 115.57 31.7499 0)
+			(at 120.65 31.7499 0)
 			(effects
 				(font
 					(size 1.27 1.27)
 				)
-				(justify right)
+				(justify left)
 			)
 		)
-		(property "Value" "R_US"
-			(at 115.57 34.2899 0)
+		(property "Value" "4k7"
+			(at 120.65 34.2899 0)
 			(effects
 				(font
 					(size 1.27 1.27)
 				)
-				(justify right)
+				(justify left)
 			)
 		)
@@
 		(fields_autoplaced yes)
 		(property "Reference" "R615"
-			(at 261.62 114.2999 0)
+			(at 266.7 114.2999 0)
 			(effects
 				(font
 					(size 1.27 1.27)
 				)
-				(justify right)
+				(justify left)
 			)
 		)
-		(property "Value" "R_US"
-			(at 261.62 116.8399 0)
+		(property "Value" "1k"
+			(at 266.7 116.8399 0)
 			(effects
 				(font
 					(size 1.27 1.27)
 				)
-				(justify right)
+				(justify left)
 			)
 		)
@@
 			)
 		)
-		(property "Value" "R_US"
-			(at 65.278 75.946 90)
+		(property "Value" "0R"
+			(at 65.024 82.55 90)
 			(effects
 				(font
@@
 		(fields_autoplaced yes)
 		(property "Reference" "R614"
-			(at 231.14 67.31 90)
+			(at 227.33 66.0399 0)
 			(effects
 				(font
 					(size 1.27 1.27)
 				)
+				(justify left)
 			)
 		)
-		(property "Value" "R_US"
-			(at 228.6 67.31 90)
+		(property "Value" "10k"
+			(at 227.33 68.5799 0)
 			(effects
 				(font
 					(size 1.27 1.27)
 				)
+				(justify left)
 			)
 		)
@@
 		(on_board yes)
 		(dnp no)
-		(fields_autoplaced yes)
 		(property "Reference" "R603"
 			(at 64.77 69.85 90)
@@
 			)
 		)
-		(property "Value" "R_US"
-			(at 64.77 72.39 90)
+		(property "Value" "0R"
+			(at 65.278 80.264 90)
 			(effects
 				(font
@@
 		(fields_autoplaced yes)
 		(property "Reference" "R608"
-			(at 115.57 48.2599 0)
+			(at 120.65 48.2599 0)
 			(effects
 				(font
 					(size 1.27 1.27)
 				)
-				(justify right)
+				(justify left)
 			)
 		)
-		(property "Value" "R_US"
-			(at 115.57 50.7999 0)
+		(property "Value" "4k7"
+			(at 120.65 50.7999 0)
 			(effects
 				(font
 					(size 1.27 1.27)
 				)
-				(justify right)
+				(justify left)
 			)
 		)
@@
 			)
 		)
-		(property "Value" "36k"
+		(property "Value" "33k"
 			(at 73.66 52.0699 0)
 			(effects
@@
 			)
 		)
-		(property "Value" "STM32F103CBTx"
+		(property "Value" "STM32F103CBT6"
 			(at 165.4967 116.84 0)
 			(effects
@@
 			)
 		)
-		(property "Value" "Crystal_GND24"
+		(property "Value" "8MHz"
 			(at 269.24 57.0798 0)
 			(effects
@@
 			)
 		)
-		(property "Value" "C"
+		(property "Value" "10uF"
 			(at 128.27 176.5299 0)
 			(effects
@@
 			)
 		)
-		(property "Value" "C"
+		(property "Value" "100nF"
 			(at 190.5 151.1299 0)
 			(effects
@@
 			)
 		)
-		(property "Value" "C"
+		(property "Value" "20pF"
 			(at 262.89 69.8499 0)
 			(effects
@@
 		(fields_autoplaced yes)
 		(property "Reference" "R613"
-			(at 222.25 67.31 90)
+			(at 218.44 66.0399 0)
 			(effects
 				(font
 					(size 1.27 1.27)
 				)
+				(justify left)
 			)
 		)
-		(property "Value" "R_US"
-			(at 219.71 67.31 90)
+		(property "Value" "DNP"
+			(at 218.44 68.5799 0)
 			(effects
 				(font
 					(size 1.27 1.27)
 				)
+				(justify left)
 			)
 		)
@@
 		(fields_autoplaced yes)
 		(property "Reference" "R616"
-			(at 261.62 148.5899 0)
+			(at 266.7 148.5899 0)
 			(effects
 				(font
 					(size 1.27 1.27)
 				)
-				(justify right)
+				(justify left)
 			)
 		)
-		(property "Value" "R_US"
-			(at 261.62 151.1299 0)
+		(property "Value" "1k"
+			(at 266.7 151.1299 0)
 			(effects
 				(font
 					(size 1.27 1.27)
 				)
-				(justify right)
+				(justify left)
 			)
 		)
@@
 			)
 		)
-		(property "Value" "USB_B_Mini"
+		(property "Value" "629105150521"
 			(at 36.83 72.3899 0)
 			(effects
@@
 			)
 		)
-		(property "Value" "C"
+		(property "Value" "100nF"
 			(at 228.6 151.1299 0)
 			(effects
@@
 			)
 		)
-		(property "Value" "C"
+		(property "Value" "20pF"
 			(at 242.57 69.8499 0)
 			(effects
@@
 			)
 		)
-		(property "Value" "C"
+		(property "Value" "10uF"
 			(at 167.64 177.7999 0)
 			(effects
@@
 			)
 		)
-		(property "Value" "C"
+		(property "Value" "100nF"
 			(at 203.2 151.1299 0)
 			(effects
@@
 			)
 		)
-		(property "Value" "C"
+		(property "Value" "100nF"
 			(at 215.9 151.1299 0)
 			(effects
@@
 		(on_board yes)
 		(dnp no)
-		(fields_autoplaced yes)
 		(property "Reference" "R601"
 			(at 64.77 64.77 90)
@@
 			)
 		)
-		(property "Value" "R_US"
-			(at 64.77 67.31 90)
+		(property "Value" "0R"
+			(at 64.77 78.486 90)
 			(effects
 				(font
@@
 			)
 		)
-		(property "Value" "R_US"
+		(property "Value" "100R"
 			(at 198.12 95.25 90)
 			(effects

Commit message: fuck. Fuck fuck. Fuck Fuck Fuck. FUUCKING FUCK
Parts:
- added R619: 1k, Resistor_SMD:R_0603_1608Metric_Pad0.98x0.95mm_HandSolder, symbol Device:R_US
- R601, R602: value 0R -> 10R
Connections:
- net at J602.3 (D+), R601.1: now also R619.2; no longer Q601.2 (E)
- new net: Q601.2 (E), R619.1
Other:
- moved on the sheet: J602
Changed lines of the file:
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@@
 	)
 	(junction
-		(at 43.18 82.55)
+		(at 38.1 82.55)
 		(diameter 0)
 		(color 0 0 0 0)
@@
 	(wire
 		(pts
-			(xy 40.64 81.28) (xy 40.64 82.55)
+			(xy 35.56 81.28) (xy 35.56 82.55)
 		)
 		(stroke
@@
 	(wire
 		(pts
-			(xy 57.15 48.26) (xy 57.15 71.12)
+			(xy 57.15 48.26) (xy 57.15 52.07)
 		)
 		(stroke
@@
 	(wire
 		(pts
-			(xy 57.15 71.12) (xy 50.8 71.12)
+			(xy 57.15 71.12) (xy 45.72 71.12)
 		)
 		(stroke
@@
 	(wire
 		(pts
-			(xy 43.18 82.55) (xy 43.18 83.82)
+			(xy 38.1 82.55) (xy 38.1 83.82)
 		)
 		(stroke
@@
 	(wire
 		(pts
-			(xy 50.8 66.04) (xy 52.07 66.04)
+			(xy 45.72 66.04) (xy 46.99 66.04)
 		)
 		(stroke
@@
 	(wire
 		(pts
-			(xy 40.64 82.55) (xy 43.18 82.55)
+			(xy 35.56 82.55) (xy 38.1 82.55)
 		)
 		(stroke
@@
 	(wire
 		(pts
-			(xy 50.8 76.2) (xy 60.96 76.2)
+			(xy 45.72 76.2) (xy 60.96 76.2)
 		)
 		(stroke
@@
 	(wire
 		(pts
-			(xy 50.8 73.66) (xy 60.96 73.66)
+			(xy 45.72 73.66) (xy 60.96 73.66)
 		)
 		(stroke
@@
 	(wire
 		(pts
+			(xy 57.15 59.69) (xy 57.15 71.12)
+		)
+		(stroke
+			(width 0)
+			(type default)
+		)
+	)
+	(wire
+		(pts
 			(xy 100.33 73.66) (xy 121.92 73.66)
 		)
@@
 	(wire
 		(pts
-			(xy 52.07 66.04) (xy 52.07 64.77)
+			(xy 46.99 66.04) (xy 46.99 64.77)
 		)
 		(stroke
@@
 	(wire
 		(pts
-			(xy 43.18 82.55) (xy 43.18 81.28)
+			(xy 38.1 82.55) (xy 38.1 81.28)
 		)
 		(stroke
@@
 	(symbol
 		(lib_id "power:VBUS")
-		(at 52.07 64.77 0)
+		(at 46.99 64.77 0)
 		(mirror y)
 		(unit 1)
@@
 		(fields_autoplaced yes)
 		(property "Reference" "#PWR0604"
-			(at 52.07 68.58 0)
+			(at 46.99 68.58 0)
 			(effects
 				(font
@@
 		)
 		(property "Value" "VBUS"
-			(at 52.07 59.69 0)
+			(at 46.99 59.69 0)
 			(effects
 				(font
@@
 		)
 		(property "Footprint" ""
-			(at 52.07 64.77 0)
+			(at 46.99 64.77 0)
 			(effects
 				(font
@@
 		)
 		(property "Datasheet" ""
-			(at 52.07 64.77 0)
+			(at 46.99 64.77 0)
 			(effects
 				(font
@@
 		)
 		(property "Description" "Power symbol creates a global label with name \"VBUS\""
-			(at 52.07 64.77 0)
+			(at 46.99 64.77 0)
 			(effects
 				(font
@@
 	(symbol
 		(lib_id "power:GND")
-		(at 43.18 83.82 0)
+		(at 38.1 83.82 0)
 		(mirror y)
 		(unit 1)
@@
 		(fields_autoplaced yes)
 		(property "Reference" "#PWR0603"
-			(at 43.18 90.17 0)
+			(at 38.1 90.17 0)
 			(effects
 				(font
@@
 		)
 		(property "Value" "GND"
-			(at 43.18 88.9 0)
+			(at 38.1 88.9 0)
 			(effects
 				(font
@@
 		)
 		(property "Footprint" ""
-			(at 43.18 83.82 0)
+			(at 38.1 83.82 0)
 			(effects
 				(font
@@
 		)
 		(property "Datasheet" ""
-			(at 43.18 83.82 0)
+			(at 38.1 83.82 0)
 			(effects
 				(font
@@
 		)
 		(property "Description" "Power symbol creates a global label with name \"GND\" , ground"
-			(at 43.18 83.82 0)
+			(at 38.1 83.82 0)
 			(effects
 				(font
@@
 		(dnp no)
 		(property "Reference" "R602"
-			(at 64.77 67.31 90)
+			(at 63.754 67.564 90)
 			(effects
 				(font
@@
 			)
 		)
-		(property "Value" "0R"
-			(at 65.024 82.55 90)
+		(property "Value" "10R"
+			(at 69.342 67.564 90)
 			(effects
 				(font
@@
 		(dnp no)
 		(property "Reference" "R603"
-			(at 64.77 69.85 90)
+			(at 61.214 78.994 90)
 			(effects
 				(font
@@
 		)
 		(property "Value" "0R"
-			(at 65.278 80.264 90)
+			(at 67.056 78.994 90)
 			(effects
 				(font
@@
 	(symbol
 		(lib_id "Connector:USB_B_Mini")
-		(at 43.18 71.12 0)
+		(at 38.1 71.12 0)
 		(unit 1)
 		(exclude_from_sim no)
@@
 		(fields_autoplaced yes)
 		(property "Reference" "J602"
-			(at 36.83 69.8499 0)
+			(at 31.75 69.8499 0)
 			(effects
 				(font
@@
 		)
 		(property "Value" "629105150521"
-			(at 36.83 72.3899 0)
+			(at 31.75 72.3899 0)
 			(effects
 				(font
@@
 		)
 		(property "Footprint" "Connector_USB:USB_Micro-B_Wuerth_629105150521"
-			(at 46.99 72.39 0)
+			(at 41.91 72.39 0)
 			(effects
 				(font
@@
 		)
 		(property "Datasheet" "~"
-			(at 46.99 72.39 0)
+			(at 41.91 72.39 0)
 			(effects
 				(font
@@
 		)
 		(property "Description" "USB Mini Type B connector"
-			(at 43.18 71.12 0)
+			(at 38.1 71.12 0)
 			(effects
 				(font
@@
 	(symbol
 		(lib_id "Device:R_US")
+		(at 57.15 55.88 0)
+		(mirror y)
+		(unit 1)
+		(exclude_from_sim no)
+		(in_bom yes)
+		(on_board yes)
+		(dnp no)
+		(fields_autoplaced yes)
+		(property "Reference" "R619"
+			(at 59.69 54.6099 0)
+			(effects
+				(font
+					(size 1.27 1.27)
+				)
+				(justify right)
+			)
+		)
+		(property "Value" "1k"
+			(at 59.69 57.1499 0)
+			(effects
+				(font
+					(size 1.27 1.27)
+				)
+				(justify right)
+			)
+		)
+		(property "Footprint" "Resistor_SMD:R_0603_1608Metric_Pad0.98x0.95mm_HandSolder"
+			(at 56.134 56.134 90)
+			(effects
+				(font
+					(size 1.27 1.27)
+				)
+				(hide yes)
+			)
+		)
+		(property "Datasheet" "~"
+			(at 57.15 55.88 0)
+			(effects
+				(font
+					(size 1.27 1.27)
+				)
+				(hide yes)
+			)
+		)
+		(property "Description" "Resistor, US symbol"
+			(at 57.15 55.88 0)
+			(effects
+				(font
+					(size 1.27 1.27)
+				)
+				(hide yes)
+			)
+		)
+		(pin "1"
+		)
+		(pin "2"
+		)
+		(instances
+			(project "Carte_moteur"
+				(path "/5d858058-eb89-4613-a7ba-0652b9f0936c/a0d73204-6cde-434c-a6b9-1c87c98088a0"
+					(reference "R619")
+					(unit 1)
+				)
+			)
+		)
+	)
+	(symbol
+		(lib_id "Device:R_US")
 		(at 196.85 34.29 0)
 		(unit 1)
@@
 		(dnp no)
 		(property "Reference" "R601"
-			(at 64.77 64.77 90)
+			(at 63.754 64.77 90)
 			(effects
 				(font
@@
 			)
 		)
-		(property "Value" "0R"
-			(at 64.77 78.486 90)
+		(property "Value" "10R"
+			(at 69.342 64.77 90)
 			(effects
 				(font
