File: Carte_power/PowkiBoard/PowkiBoard.kicad_sch (KiCad schematic)
At the start: 75 parts, among them J1 AUConn, J2 VBATT, J3 GNDBATT

Commit message: AAAAAAAAAAAAAAAA
Parts:
- U1, U2, U3: footprint Package_DFN_QFN:WDFN-10-1EP_3x3mm_P0.5mm_EP1.8x2.5mm -> Devices:RTQ6365
Changed lines of the file:
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@@
 			)
 		)
-		(property "Footprint" "Package_DFN_QFN:WDFN-10-1EP_3x3mm_P0.5mm_EP1.8x2.5mm"
+		(property "Footprint" "Devices:RTQ6365"
 			(at 121.92 93.98 0)
 			(effects
@@
 			)
 		)
-		(property "Footprint" "Package_DFN_QFN:WDFN-10-1EP_3x3mm_P0.5mm_EP1.8x2.5mm"
+		(property "Footprint" "Devices:RTQ6365"
 			(at 121.92 46.99 0)
 			(effects
@@
 			)
 		)
-		(property "Footprint" "Package_DFN_QFN:WDFN-10-1EP_3x3mm_P0.5mm_EP1.8x2.5mm"
+		(property "Footprint" "Devices:RTQ6365"
 			(at 121.92 138.43 0)
 			(effects
