File: Carte_power/PowkiBoard/logic_converter.kicad_sch (KiCad schematic)
At the start: 23 parts, among them J8 SWLogic

Commit message: AAAAAAAAAAAAAAAA
Parts:
- U4: footprint Package_DFN_QFN:WDFN-10-1EP_3x3mm_P0.5mm_EP1.8x2.5mm -> Devices:RTQ6365
Changed lines of the file:
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@@
 			)
 		)
-		(property "Footprint" "Package_DFN_QFN:WDFN-10-1EP_3x3mm_P0.5mm_EP1.8x2.5mm"
+		(property "Footprint" "Devices:RTQ6365"
 			(at 137.16 96.52 0)
 			(effects
