File: Carte_interco_H7/Interco_weactH7/Interco_weactH7.kicad_sch (KiCad schematic)
At the start: 43 parts, among them J101 servo orientation, J102 servo bras, J103 servo dicristaline, J104 servo dicristaline, J105 POW_access, J106 KK-254_AE-6410-07A, J107 LIDAR, J108 LIDAR, J109 SNDBOARD, J110 electroaimant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

Commit message: WIP. layout ok
Parts:
- removed C102, C107: 100n, Capacitor_SMD:C_1206_3216Metric_Pad1.33x1.80mm_HandSolder, symbol Device:C
- removed D101, D102, D103: 1N4007, Diode_THT:D_DO-41_SOD81_P10.16mm_Horizontal, symbol Diode:1N4007
- removed J110: electroaimant, Connector_Molex:Molex_KK-254_AE-6410-02A_1x02_P2.54mm_Vertical, symbol Connector:Conn_01x02_Female
- removed J111: SWrobot, Connector_Molex:Molex_KK-254_AE-6410-02A_1x02_P2.54mm_Vertical, symbol Connector:Conn_01x02_Female
- removed J113: pompe, Connector_Molex:Molex_KK-254_AE-6410-02A_1x02_P2.54mm_Vertical, symbol Connector:Conn_01x02_Female
- removed Q101, Q102: SW_pompe, Package_TO_SOT_THT:TO-220-3_Vertical, symbol Device:Q_NMOS_GDS
- removed Q103: SW_vanne, Package_TO_SOT_THT:TO-220-3_Vertical, symbol Device:Q_NMOS_GDS
- removed R101, R102, R105, R106: 330, Capacitor_SMD:C_0805_2012Metric_Pad1.18x1.45mm_HandSolder, symbol Device:R
- removed R103, R104, R107, R108: 1k, Capacitor_SMD:C_0805_2012Metric_Pad1.18x1.45mm_HandSolder, symbol Device:R
- added C109, C110: 100n, Capacitor_SMD:C_1206_3216Metric_Pad1.33x1.80mm_HandSolder, symbol Device:C
- added J110, J118: servo orientation, Connector_Molex:Molex_KK-254_AE-6410-03A_1x03_P2.54mm_Vertical, symbol Connector:Conn_01x03_Male
- added J111, J119: servo bras, Connector_Molex:Molex_KK-254_AE-6410-03A_1x03_P2.54mm_Vertical, symbol Connector:Conn_01x03_Male
- added J120: SWrobot, Connector_Molex:Molex_KK-254_AE-6410-02A_1x02_P2.54mm_Vertical, symbol Connector:Conn_01x02_Female
- added J121: reset, Connector_Molex:Molex_KK-254_AE-6410-02A_1x02_P2.54mm_Vertical, symbol Connector:Conn_01x02_Female
- J105: footprint Connector_Molex:Molex_Nano-Fit_105314-xx08_2x04_P2.50mm_Horizontal -> Connector_Molex:Molex_Nano-Fit_105310-xx08_2x04_P2.50mm_Vertical
- J116: value vanne -> SWcote
Connections:
- net +5V_PWR: now also C109.1, C110.1, J110.2 (Pin_2), J111.2 (Pin_2), J118.2 (Pin_2), J119.2 (Pin_2)
- net GND: now also J112.2 (Pin_2), J114.2 (Pin_2), J115.2 (Pin_2), J116.2 (Pin_2), C109.2, C110.2, J110.1 (Pin_1), J111.1 (Pin_1), J118.1 (Pin_1), J119.1 (Pin_1), J120.2 (Pin_2), J121.2 (Pin_2)
- net WEACT/IO6: now reaches J116.1 (Pin_1)
- removed net SW_3V3: J112.1 (Pin_1), J114.1 (Pin_1), J115.1 (Pin_1)
- new net PWM_SERVO5: J118.3 (Pin_3)
- new net PWM_SERVO6: J119.3 (Pin_3)
- new net WEACT/IO1: J121.1 (Pin_1)
- new net WEACT/IO2: J115.1 (Pin_1)
- new net WEACT/IO3: J120.1 (Pin_1)
- new net WEACT/IO4: J112.1 (Pin_1)
- new net WEACT/IO5: J114.1 (Pin_1)
Other:
- sheet WEACT ports: added IO1, IO2, IO3, IO4, IO5, IO6, SERVO5, SERVO6; removed none
- note removed: "hydrolique"
- moved on the sheet: C101, C103, C104, C105, C106, J101, J102, J103, J104, J112, J114, J115

Commit message: ready for check
Connections:
- net WEACT/IO8: now reaches J111.3 (Pin_3)
- net WEACT/IO7: now reaches J110.3 (Pin_3)
- no-connect marks 0 -> 8
Other:
- sheet WEACT ports: added IO7, IO8; removed none
- sheet stlink ports: added none; removed 5V_EXT
- moved on the sheet: J105
