File: Carte_interco_H7/Interco_weactH7/Interco_weactH7.kicad_sch (KiCad schematic)
At the start: 32 parts, among them J101 servo orientation, J102 servo bras, J103 servo dicristaline, J104 servo dicristaline, J105 POW_access, J106 KK-254_AE-6410-07A, J107 LIDAR, J108 LIDAR, J109 SNDBOARD, J110 servo orientation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

Commit message: send PCB
Parts:
- C101, C103, C104, C105, C106, C108, C109, C110: value 100n -> 10uF; DK_PN (none) -> 490-GRM21BZ71E106KE15LCT-ND; Size (none) -> 1206
- H101, H102, H103, H104: now not fitted
- J101, J102, J103, J104, J110, J111, J118, J119: DK_PN (none) -> 281695-3
- J105: DK_PN (none) -> WM16881-ND
- J106: DK_PN (none) -> WM4116-ND
- J107, J108: DK_PN (none) -> WM4113-ND
- J109: DK_PN (none) -> WM4114-ND
- J114, J115, J116, J120, J121: DK_PN (none) -> 0022232021
- U101: DK_PN (none) -> 497-1242-1-ND
