File: Carte_interco_H7/Interco_weactH7/WeAct.kicad_sch (KiCad schematic)
At the start: 13 parts

Commit message: ready for check
Connections:
- net GND: now also U201.P1_1 (GND), U201.P2_1 (GND), U201.P2_15 (GND)
- net SERVO1: now also U201.P1_36 (PD12); no longer U201.P2_32 (PE9)
- net SERVO2: now also U201.P1_35 (PD13); no longer U201.P2_34 (PE11)
- net SERVO3: now also U201.P1_34 (PD14); no longer U201.P2_36 (PE13)
- net SERVO4: now also U201.P1_33 (PD15); no longer U201.P2_37 (PE14)
- net UART7_RX: now also R202.1
- net UART7_TX: now also R201.1
- net UNICORN_RST: now also U201.P1_44 (PB12); no longer U201.P2_38 (PE15)
- net UNICORN_RX(MI): now also U201.P1_41 (PB15); no longer U201.P2_40 (PB11)
- net UNICORN_TX(MO): now also U201.P1_42 (PB14); no longer U201.P2_39 (PB10)
- net SERVO5: now reaches U201.P1_10 (PB4)
- net IO8: now reaches U201.P1_14 (PD5)
- net IO7: now reaches U201.P1_16 (PD3)
- net IO1: now reaches U201.P1_3 (PE1)
- net IO4: now reaches U201.P1_4 (PE0)
- net IO2: now reaches U201.P1_5 (PB9)
- net IO5: now reaches U201.P1_6 (PB8)
- net IO3: now reaches U201.P1_7 (PB7)
- net IO6: now reaches U201.P1_8 (PB6)
- net SERVO6: now reaches U201.P1_9 (PB5)
- net UART5_RX renamed USART3_RX
- net USART3_RX: now also U201.P2_40 (PB11); no longer U201.P1_44 (PB12)
- net UART5_TX: no longer names the net of U201.P1_43 (PB13)
- net UART5_TX: no longer R203.1
- removed net USART1_RX: R202.1, U201.P1_41 (PB15)
- removed net USART1_TX: R201.1, U201.P1_42 (PB14)
- new net USART3_TX: R203.1, U201.P2_39 (PB10)
- no-connect marks 0 -> 41
Other:
- moved on the sheet: U201C
