File: Carte_interco_H7/Interco_weactH7/WeAct.kicad_sch (KiCad schematic)
At the start: 13 parts

Commit message: pins in conflict rerouted
Connections:
- net SERVO1: now also U201.P1_34 (PD14); no longer U201.P1_28 (PA8)
- net SERVO2: now also U201.P1_33 (PD15); no longer U201.P1_27 (PA9)
- net SERVO3: now also U201.P1_29 (PC9); no longer U201.P1_34 (PD14)
- net SERVO4: now also U201.P1_27 (PA9); no longer U201.P1_33 (PD15)
- net SERVO5: now also U201.P1_9 (PB5); no longer U201.P1_29 (PC9)
- net SERVO6: now also U201.P1_28 (PA8); no longer U201.P1_9 (PB5)
Changed lines of the file:
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@@
+		)
+	)
+	(label "TIM4_CH4"
+		(at 81.28 129.54 0)
+		(effects
+			(font
+				(size 1.27 1.27)
+			)
+			(justify left bottom)
 		)
 	)
@@
 		)
 	)
-	(label "TIM1_CH2"
-		(at 81.28 129.54 0)
-		(effects
-			(font
-				(size 1.27 1.27)
-			)
-			(justify left bottom)
-		)
-	)
 	(label "DBG2"
 		(at 233.68 33.02 180)
@@
 		)
 	)
-	(label "TIM4_CH4"
-		(at 81.28 139.7 0)
-		(effects
-			(font
-				(size 1.27 1.27)
-			)
-			(justify left bottom)
-		)
-	)
-	(label "TIM3_CH2"
-		(at 81.28 149.86 0)
-		(effects
-			(font
-				(size 1.27 1.27)
-			)
-			(justify left bottom)
-		)
-	)
 	(label "USART6_TX"
 		(at 119.38 58.42 180)
@@
 		)
 	)
-	(label "TIM4_CH3"
-		(at 81.28 134.62 0)
-		(effects
-			(font
-				(size 1.27 1.27)
-			)
-			(justify left bottom)
-		)
-	)
 	(label "SPI3_MISO"
 		(at 62.23 45.72 0)
@@
 		)
 	)
+	(label "TIM1_CH1"
+		(at 81.28 149.86 0)
+		(effects
+			(font
+				(size 1.27 1.27)
+			)
+			(justify left bottom)
+		)
+	)
 	(label "USART1_TX"
 		(at 129.54 156.21 0)
@@
 		)
 	)
+	(label "TIM3_CH4"
+		(at 81.28 134.62 0)
+		(effects
+			(font
+				(size 1.27 1.27)
+			)
+			(justify left bottom)
+		)
+	)
 	(label "PE1"
 		(at 62.23 22.86 0)
@@
 		)
 	)
+	(label "TIM4_CH3"
+		(at 81.28 124.46 0)
+		(effects
+			(font
+				(size 1.27 1.27)
+			)
+			(justify left bottom)
+		)
+	)
 	(label "USART2_TX"
 		(at 161.29 43.18 0)
@@
 		)
 	)
-	(label "TIM1_CH1"
-		(at 81.28 124.46 0)
-		(effects
-			(font
-				(size 1.27 1.27)
-			)
-			(justify left bottom)
-		)
-	)
 	(label "TIM1_CH2"
 		(at 62.23 53.34 0)
@@
 		)
 	)
-	(label "TIM3_CH4"
-		(at 81.28 144.78 0)
+	(label "TIM1_CH2"
+		(at 81.28 139.7 0)
 		(effects
 			(font
@@
 		(effects
 			(font
+				(size 1.27 1.27)
+			)
+			(justify left bottom)
+		)
+	)
+	(label "TIM3_CH2"
+		(at 81.28 144.78 0)
+		(effects
+			(font

Commit message: send PCB
Parts:
- D201, D202: value LED -> LED_GREEN; DK_PN (none) -> L62505CT-ND
- D203, D204: value LED -> LED_RED; DK_PN (none) -> L62501CT-ND
- R201, R202, R203, R204: value R_US -> JUMPER; DK_PN (none) -> 541-0.0GCT-ND; Size (none) -> 0805
- R205, R206, R207, R208: DK_PN (none) -> 311-1.00KHRCT-ND; Size (none) -> 0603
Connections:
- net SERVO1: now also U201.P1_33 (PD15); no longer U201.P1_34 (PD14)
- net SERVO2: now also U201.P1_34 (PD14); no longer U201.P1_33 (PD15)
Changed lines of the file:
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@@
 		)
 	)
-	(label "TIM4_CH4"
-		(at 81.28 129.54 0)
-		(effects
-			(font
-				(size 1.27 1.27)
-			)
-			(justify left bottom)
-		)
-	)
 	(label "UART7_RX"
 		(at 233.68 55.88 180)
@@
 		)
 	)
+	(label "TIM4_CH3"
+		(at 81.28 129.54 0)
+		(effects
+			(font
+				(size 1.27 1.27)
+			)
+			(justify left bottom)
+		)
+	)
 	(label "PA4"
 		(at 22.86 153.67 0)
@@
 		)
 	)
+	(label "TIM4_CH4"
+		(at 81.28 124.46 0)
+		(effects
+			(font
+				(size 1.27 1.27)
+			)
+			(justify left bottom)
+		)
+	)
 	(label "TIM2_CH1"
 		(at 233.68 45.72 180)
@@
 		)
 	)
-	(label "TIM4_CH3"
-		(at 81.28 124.46 0)
-		(effects
-			(font
-				(size 1.27 1.27)
-			)
-			(justify left bottom)
-		)
-	)
 	(label "USART2_TX"
 		(at 161.29 43.18 0)
@@
 			)
 		)
-		(property "Value" "LED"
+		(property "Value" "LED_RED"
 			(at 261.62 153.9874 90)
 			(effects
@@
 			)
 		)
+		(property "DK_PN" "L62501CT-ND"
+			(at 257.81 151.13 0)
+			(effects
+				(font
+					(size 1.27 1.27)
+				)
+			)
+		)
 		(pin "1"
 		)
@@
 			)
 		)
-		(property "Value" "R_US"
+		(property "Value" "JUMPER"
 			(at 41.91 130.81 90)
 			(effects
@@
 			)
 		)
+		(property "DK_PN" "541-0.0GCT-ND"
+			(at 41.91 134.62 0)
+			(effects
+				(font
+					(size 1.27 1.27)
+				)
+			)
+		)
+		(property "Size" "0805"
+			(at 41.91 134.62 0)
+			(effects
+				(font
+					(size 1.27 1.27)
+				)
+			)
+		)
 		(pin "1"
 		)
@@
 			)
 		)
+		(property "DK_PN" "311-1.00KHRCT-ND"
+			(at 245.11 142.24 0)
+			(effects
+				(font
+					(size 1.27 1.27)
+				)
+			)
+		)
+		(property "Size" "0603"
+			(at 245.11 142.24 0)
+			(effects
+				(font
+					(size 1.27 1.27)
+				)
+			)
+		)
 		(pin "1"
 		)
@@
 			)
 		)
+		(property "DK_PN" "311-1.00KHRCT-ND"
+			(at 232.41 142.24 0)
+			(effects
+				(font
+					(size 1.27 1.27)
+				)
+			)
+		)
+		(property "Size" "0603"
+			(at 232.41 142.24 0)
+			(effects
+				(font
+					(size 1.27 1.27)
+				)
+			)
+		)
 		(pin "1"
 		)
@@
 			)
 		)
-		(property "Value" "LED"
+		(property "Value" "LED_GREEN"
 			(at 236.22 153.9874 90)
 			(effects
@@
 			)
 		)
+		(property "DK_PN" "L62505CT-ND"
+			(at 232.41 151.13 0)
+			(effects
+				(font
+					(size 1.27 1.27)
+				)
+			)
+		)
 		(pin "1"
 		)
@@
 			)
 		)
+		(property "DK_PN" "311-1.00KHRCT-ND"
+			(at 257.81 142.24 0)
+			(effects
+				(font
+					(size 1.27 1.27)
+				)
+			)
+		)
+		(property "Size" "0603"
+			(at 257.81 142.24 0)
+			(effects
+				(font
+					(size 1.27 1.27)
+				)
+			)
+		)
 		(pin "1"
 		)
@@
 			)
 		)
-		(property "Value" "R_US"
+		(property "Value" "JUMPER"
 			(at 41.91 161.29 90)
 			(effects
@@
 			)
 		)
+		(property "DK_PN" "541-0.0GCT-ND"
+			(at 41.91 165.1 0)
+			(effects
+				(font
+					(size 1.27 1.27)
+				)
+			)
+		)
+		(property "Size" "0805"
+			(at 41.91 165.1 0)
+			(effects
+				(font
+					(size 1.27 1.27)
+				)
+			)
+		)
 		(pin "1"
 		)
@@
 			)
 		)
-		(property "Value" "R_US"
+		(property "Value" "JUMPER"
 			(at 41.91 139.7 90)
 			(effects
@@
 			)
 		)
+		(property "DK_PN" "541-0.0GCT-ND"
+			(at 41.91 143.51 0)
+			(effects
+				(font
+					(size 1.27 1.27)
+				)
+			)
+		)
+		(property "Size" "0805"
+			(at 41.91 143.51 0)
+			(effects
+				(font
+					(size 1.27 1.27)
+				)
+			)
+		)
 		(pin "1"
 		)
@@
 			)
 		)
+		(property "DK_PN" ""
+			(at 205.74 156.21 0)
+			(effects
+				(font
+					(size 1.27 1.27)
+				)
+			)
+		)
 		(pin "D3"
 		)
@@
 			)
 		)
-		(property "Value" "R_US"
+		(property "Value" "JUMPER"
 			(at 41.91 170.18 90)
 			(effects
@@
 			)
 		)
+		(property "DK_PN" "541-0.0GCT-ND"
+			(at 41.91 173.99 0)
+			(effects
+				(font
+					(size 1.27 1.27)
+				)
+			)
+		)
+		(property "Size" "0805"
+			(at 41.91 173.99 0)
+			(effects
+				(font
+					(size 1.27 1.27)
+				)
+			)
+		)
 		(pin "1"
 		)
@@
 			)
 		)
+		(property "DK_PN" ""
+			(at 196.85 77.47 0)
+			(effects
+				(font
+					(size 1.27 1.27)
+				)
+			)
+		)
 		(pin "D3"
 		)
@@
 			)
 		)
+		(property "DK_PN" ""
+			(at 91.44 77.47 0)
+			(effects
+				(font
+					(size 1.27 1.27)
+				)
+			)
+		)
 		(pin "D3"
 		)
@@
 			)
 		)
+		(property "DK_PN" "311-1.00KHRCT-ND"
+			(at 269.24 142.24 0)
+			(effects
+				(font
+					(size 1.27 1.27)
+				)
+			)
+		)
+		(property "Size" "0603"
+			(at 269.24 142.24 0)
+			(effects
+				(font
+					(size 1.27 1.27)
+				)
+			)
+		)
 		(pin "1"
 		)
@@
 			)
 		)
-		(property "Value" "LED"
+		(property "Value" "LED_GREEN"
 			(at 248.92 153.9874 90)
 			(effects
@@
 			)
 		)
+		(property "DK_PN" "L62505CT-ND"
+			(at 245.11 151.13 0)
+			(effects
+				(font
+					(size 1.27 1.27)
+				)
+			)
+		)
 		(pin "1"
 		)
@@
 			)
 		)
-		(property "Value" "LED"
+		(property "Value" "LED_RED"
 			(at 273.05 153.9874 90)
 			(effects
@@
 			)
 		)
+		(property "DK_PN" "L62501CT-ND"
+			(at 269.24 151.13 0)
+			(effects
+				(font
+					(size 1.27 1.27)
+				)
+			)
+		)
