File: Carte_interco_H7/Interco_weactH7/stlink.kicad_sch (KiCad schematic)
At the start: 38 parts, among them J117 Conn_02x07_Odd_Even, J301 629105150521, J302 Conn_01x06_Pin, Q301 MMBTA44, U301 ECMF02-2AMX6, U302 LD1117S33TR_SOT223, U303 STM32F103CBT6, Y301 8MHz

Commit message: ready for check
Parts:
- removed D303: PMEG40T10ER, Diode_SMD:Nexperia_CFP3_SOD-123W, symbol Diode:PMEG40T10ER
Changed lines of the file:
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@@
 	(wire
 		(pts
-			(xy 73.66 102.87) (xy 80.01 102.87)
-		)
-		(stroke
-			(width 0)
-			(type default)
-		)
-	)
-	(wire
-		(pts
 			(xy 119.38 114.3) (xy 119.38 118.11)
 		)
@@
 	(wire
 		(pts
-			(xy 80.01 102.87) (xy 80.01 114.3)
-		)
-		(stroke
-			(width 0)
-			(type default)
-		)
-	)
-	(wire
-		(pts
 			(xy 83.82 166.37) (xy 81.28 166.37)
 		)
@@
 	(wire
 		(pts
-			(xy 63.5 102.87) (xy 66.04 102.87)
-		)
-		(stroke
-			(width 0)
-			(type default)
-		)
-	)
-	(wire
-		(pts
 			(xy 45.72 66.04) (xy 45.72 114.3)
 		)
@@
 		)
 	)
-	(hierarchical_label "5V_EXT"
-		(shape input)
-		(at 63.5 102.87 180)
-		(effects
-			(font
-				(size 1.27 1.27)
-			)
-			(justify right)
-		)
-	)
 	(hierarchical_label "STLINK_RX"
 		(shape input)
@@
 					(unit 1)
 				)
-			)
-		)
-	)
-	(symbol
-		(lib_id "Diode:PMEG40T10ER")
-		(at 69.85 102.87 180)
-		(unit 1)
-		(exclude_from_sim no)
-		(in_bom yes)
-		(on_board yes)
-		(dnp no)
-		(fields_autoplaced yes)
-		(property "Reference" "D303"
-			(at 70.1675 96.52 0)
-			(effects
-				(font
-					(size 1.27 1.27)
-				)
-			)
-		)
-		(property "Value" "PMEG40T10ER"
-			(at 70.1675 99.06 0)
-			(effects
-				(font
-					(size 1.27 1.27)
-				)
-			)
-		)
-		(property "Footprint" "Diode_SMD:Nexperia_CFP3_SOD-123W"
-			(at 69.85 98.425 0)
-			(effects
-				(font
-					(size 1.27 1.27)
-				)
-				(hide yes)
-			)
-		)
-		(property "Datasheet" "https://assets.nexperia.com/documents/data-sheet/PMEG40T10ER.pdf"
-			(at 69.85 102.87 0)
-			(effects
-				(font
-					(size 1.27 1.27)
-				)
-				(hide yes)
-			)
-		)
-		(property "Description" "40V, 1A low Vf Trench MEGA Schottky barrier rectifier, SOD-123W"
-			(at 69.85 102.87 0)
-			(effects
-				(font
-					(size 1.27 1.27)
-				)
-				(hide yes)
-			)
-		)
-		(pin "1"
-		)
-		(pin "2"
-		)
-		(instances
-			(project "Carte_moteur"
-				(path "/5d858058-eb89-4613-a7ba-0652b9f0936c/a0d73204-6cde-434c-a6b9-1c87c98088a0"
-					(reference "D601")
-					(unit 1)
-				)
-			)
-			(project "Carte_moteur"
-				(path "/e63e39d7-6ac0-4ffd-8aa3-1841a4541b55/b744349d-9aa8-4cc0-b442-5d75bd8e239a"
-					(reference "D303")
-					(unit 1)
-				)

Commit message: send PCB
Parts:
- C301, C302: DK_PN (none) -> 490-GRM21BZ71E106KE15LCT-ND
- C303, C304, C306, C307: DK_PN (none) -> 399-C0603C104K5RAC7411CT-ND
- C305: value C -> 1nF; DK_PN (none) -> C0603X102K5RAC3316
- C308, C309: DK_PN (none) -> 1276-1187-1-ND
- D302, D304: DK_PN (none) -> 1727-7478-1-ND
- D305: value LED -> LED_RED; DK_PN (none) -> L62501CT-ND
- D306: value LED -> LED_GREEN; DK_PN (none) -> L62505CT-ND
- J117, J302: now not fitted
- J301: DK_PN (none) -> 732-5960-1-ND
- Q301: DK_PN (none) -> 4878-MMBTA44CT-ND
- R301, R316, R317: DK_PN (none) -> 311-1.00KHRCT-ND; Size (none) -> 0603
- R302, R303: DK_PN (none) -> RMCF0603FT10R0CT-ND; Size (none) -> 0603
- R305, R315: DK_PN (none) -> 2019-RK73H1JTTD1002FCT-ND; Size (none) -> 0603
- R306: DK_PN (none) -> 311-33.0KHRCT-ND; Size (none) -> 0603
- R307, R312: DK_PN (none) -> 311-100HRCT-ND; Size (none) -> 0603
- R308, R309: value 4k7 -> 10k; DK_PN (none) -> 2019-RK73H1JTTD1002FCT-ND; Size (none) -> 0603
- R310, R311, R313: value R_US -> 10k; DK_PN (none) -> 2019-RK73H1JTTD1002FCT-ND; Size (none) -> 0603
- R314: Size (none) -> 0603; now not fitted
- U301: DK_PN (none) -> 497-10773-1-ND
- U302: DK_PN (none) -> 497-1242-1-ND
- U303: DK_PN (none) -> 497-17380-1-ND
- Y301: DK_PN (none) -> 1923-830059082CT-ND
