File: Carte_interco_H7/Interco_weactH7/tmc.kicad_sch (KiCad schematic)
At the start: 16 parts, among them J401 KK-254_AE-6410-04A, J402 KK-254_AE-6410-04A, U401 TMC2209, U402 TMC2209

Commit message: send PCB
Parts:
- C401, C403: value 47uF -> 22uF; DK_PN (none) -> 587-5481-1-ND
- C402, C404: DK_PN (none) -> 490-GRM21BZ71E106KE15LCT-ND
- J401, J402: DK_PN (none) -> WM4113-ND
- R401, R402, R403, R404, R405, R406, R407, R408: value R_US -> JUMPER; DK_PN (none) -> 541-0.0GCT-ND; Size (none) -> 0805
- U401, U402: DK_PN (none) -> 801-87-032-10-012101
Changed lines of the file:
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@@
 		(polyline
 			(pts
-				(xy 168.91 116.84) (xy 171.45 116.84) (xy 171.45 129.54) (xy 168.91 129.54)
+				(xy 168.91 57.15) (xy 171.45 57.15) (xy 171.45 69.85) (xy 168.91 69.85)
 			)
 			(stroke
@@
 		(polyline
 			(pts
-				(xy 168.91 57.15) (xy 171.45 57.15) (xy 171.45 69.85) (xy 168.91 69.85)
+				(xy 168.91 116.84) (xy 171.45 116.84) (xy 171.45 129.54) (xy 168.91 129.54)
 			)
 			(stroke
@@
 			)
 		)
+		(property "DK_PN" "WM4113-ND"
+			(at 214.63 123.19 0)
+			(effects
+				(font
+					(size 1.27 1.27)
+				)
+				(hide yes)
+			)
+		)
 		(pin "1"
 		)
@@
 			)
 		)
-		(property "Value" "R_US"
+		(property "Value" "JUMPER"
 			(at 77.47 49.53 90)
 			(effects
@@
 			)
 		)
+		(property "DK_PN" "541-0.0GCT-ND"
+			(at 81.28 49.53 0)
+			(effects
+				(font
+					(size 1.27 1.27)
+				)
+				(hide yes)
+			)
+		)
+		(property "Size" "0805"
+			(at 81.28 49.53 0)
+			(effects
+				(font
+					(size 1.27 1.27)
+				)
+				(hide yes)
+			)
+		)
 		(pin "1"
 		)
@@
 			)
 		)
-		(property "Value" "R_US"
+		(property "Value" "JUMPER"
 			(at 77.47 125.73 90)
 			(effects
@@
 			)
 		)
+		(property "DK_PN" "541-0.0GCT-ND"
+			(at 81.28 125.73 0)
+			(effects
+				(font
+					(size 1.27 1.27)
+				)
+				(hide yes)
+			)
+		)
+		(property "Size" "0805"
+			(at 81.28 125.73 0)
+			(effects
+				(font
+					(size 1.27 1.27)
+				)
+				(hide yes)
+			)
+		)
 		(pin "1"
 		)
@@
 			)
 		)
+		(property "DK_PN" "490-GRM21BZ71E106KE15LCT-ND"
+			(at 151.13 176.53 0)
+			(effects
+				(font
+					(size 1.27 1.27)
+				)
+				(hide yes)
+			)
+		)
 		(pin "1"
 		)
@@
 			)
 		)
-		(property "Value" "47uF"
+		(property "Value" "22uF"
 			(at 87.63 177.7999 0)
 			(effects
@@
 			)
 		)
+		(property "DK_PN" "587-5481-1-ND"
+			(at 83.82 176.53 0)
+			(effects
+				(font
+					(size 1.27 1.27)
+				)
+				(hide yes)
+			)
+		)
 		(pin "2"
 		)
@@
 			)
 		)
-		(property "Value" "R_US"
+		(property "Value" "JUMPER"
 			(at 87.63 49.53 90)
 			(effects
@@
 			)
 		)
+		(property "DK_PN" "541-0.0GCT-ND"
+			(at 91.44 49.53 0)
+			(effects
+				(font
+					(size 1.27 1.27)
+				)
+				(hide yes)
+			)
+		)
+		(property "Size" "0805"
+			(at 91.44 49.53 0)
+			(effects
+				(font
+					(size 1.27 1.27)
+				)
+				(hide yes)
+			)
+		)
 		(pin "1"
 		)
@@
 			)
 		)
+		(property "DK_PN" "801-87-032-10-012101"
+			(at 151.13 60.96 0)
+			(effects
+				(font
+					(size 1.27 1.27)
+				)
+				(hide yes)
+			)
+		)
 		(pin "5"
 		)
@@
 			)
 		)
-		(property "Value" "R_US"
+		(property "Value" "JUMPER"
 			(at 77.47 66.04 90)
 			(effects
@@
 			)
 		)
+		(property "DK_PN" "541-0.0GCT-ND"
+			(at 81.28 66.04 0)
+			(effects
+				(font
+					(size 1.27 1.27)
+				)
+				(hide yes)
+			)
+		)
+		(property "Size" "0805"
+			(at 81.28 66.04 0)
+			(effects
+				(font
+					(size 1.27 1.27)
+				)
+				(hide yes)
+			)
+		)
 		(pin "1"
 		)
@@
 			)
 		)
-		(property "Value" "R_US"
+		(property "Value" "JUMPER"
 			(at 87.63 125.73 90)
 			(effects
@@
 			)
 		)
+		(property "DK_PN" "541-0.0GCT-ND"
+			(at 91.44 125.73 0)
+			(effects
+				(font
+					(size 1.27 1.27)
+				)
+				(hide yes)
+			)
+		)
+		(property "Size" "0805"
+			(at 91.44 125.73 0)
+			(effects
+				(font
+					(size 1.27 1.27)
+				)
+				(hide yes)
+			)
+		)
 		(pin "1"
 		)
@@
 			)
 		)
-		(property "Value" "R_US"
+		(property "Value" "JUMPER"
 			(at 87.63 66.04 90)
 			(effects
@@
 			)
 		)
+		(property "DK_PN" "541-0.0GCT-ND"
+			(at 91.44 66.04 0)
+			(effects
+				(font
+					(size 1.27 1.27)
+				)
+				(hide yes)
+			)
+		)
+		(property "Size" "0805"
+			(at 91.44 66.04 0)
+			(effects
+				(font
+					(size 1.27 1.27)
+				)
+				(hide yes)
+			)
+		)
 		(pin "1"
 		)
@@
 			)
 		)
+		(property "DK_PN" "801-87-032-10-012101"
+			(at 151.13 120.65 0)
+			(effects
+				(font
+					(size 1.27 1.27)
+				)
+				(hide yes)
+			)
+		)
 		(pin "5"
 		)
@@
 			)
 		)
-		(property "Value" "47uF"
+		(property "Value" "22uF"
 			(at 133.35 177.7999 0)
 			(effects
@@
 			)
 		)
+		(property "DK_PN" "587-5481-1-ND"
+			(at 129.54 176.53 0)
+			(effects
+				(font
+					(size 1.27 1.27)
+				)
+				(hide yes)
+			)
+		)
 		(pin "2"
 		)
@@
 			)
 		)
-		(property "Value" "R_US"
+		(property "Value" "JUMPER"
 			(at 87.63 109.22 90)
 			(effects
@@
 			)
 		)
+		(property "DK_PN" "541-0.0GCT-ND"
+			(at 91.44 109.22 0)
+			(effects
+				(font
+					(size 1.27 1.27)
+				)
+				(hide yes)
+			)
+		)
+		(property "Size" "0805"
+			(at 91.44 109.22 0)
+			(effects
+				(font
+					(size 1.27 1.27)
+				)
+				(hide yes)
+			)
+		)
 		(pin "1"
 		)
@@
 			)
 		)
+		(property "DK_PN" "490-GRM21BZ71E106KE15LCT-ND"
+			(at 105.41 176.53 0)
+			(effects
+				(font
+					(size 1.27 1.27)
+				)
+				(hide yes)
+			)
+		)
 		(pin "1"
 		)
@@
 			)
 		)
+		(property "DK_PN" "WM4113-ND"
+			(at 214.63 63.5 0)
+			(effects
+				(font
+					(size 1.27 1.27)
+				)
+				(hide yes)
+			)
+		)
 		(pin "1"
 		)
@@
 			)
 		)
-		(property "Value" "R_US"
+		(property "Value" "JUMPER"
 			(at 77.47 109.22 90)
 			(effects
@@
 			(at 81.28 109.22 0)
 			(effects
+				(font
+					(size 1.27 1.27)
+				)
+				(hide yes)
+			)
+		)
+		(property "DK_PN" "541-0.0GCT-ND"
+			(at 81.28 109.22 0)
+			(effects
+				(font
+					(size 1.27 1.27)
+				)
+				(hide yes)
+			)
+		)
+		(property "Size" "0805"
+			(at 81.28 109.22 0)
+			(effects
